File: pcb/PiPLC-HMI/PiPLC-HMI.kicad_sch (KiCad schematic)
At the start: 23 parts, among them J1 Conn_02x12_Odd_Even, J2 KNX, J3 Wago Pin Header 1mm, J4 Wago Pin Header 1mm

Commit message: [HMI] Flip pin assignment of boardboard interface
Connections:
- net +3V3: now also J1.7 (Pin_7); no longer J1.8 (Pin_8)
- net GND: now also J1.4 (Pin_4); no longer J1.3 (Pin_3)
- net KNX +: now also J1.8 (Pin_8); no longer J1.7 (Pin_7)
- net KNX -: now also J1.6 (Pin_6); no longer J1.5 (Pin_5)
- net LED_24V: now also J1.3 (Pin_3); no longer J1.4 (Pin_4)
- net LED_5V: now also J1.5 (Pin_5); no longer J1.6 (Pin_6)
- net LED_I1: now also J1.9 (Pin_9); no longer J1.10 (Pin_10)
- net LED_I2: now also J1.11 (Pin_11); no longer J1.12 (Pin_12)
- net LED_I3: now also J1.13 (Pin_13); no longer J1.14 (Pin_14)
- net LED_I4: now also J1.15 (Pin_15); no longer J1.16 (Pin_16)
- net LED_I5: now also J1.17 (Pin_17); no longer J1.18 (Pin_18)
- net LED_I6: now also J1.19 (Pin_19); no longer J1.20 (Pin_20)
- net LED_I7: now also J1.21 (Pin_21); no longer J1.22 (Pin_22)
- net LED_I8: now also J1.23 (Pin_23); no longer J1.24 (Pin_24)
- net LED_Q1: now also J1.24 (Pin_24); no longer J1.23 (Pin_23)
- net LED_Q2: now also J1.22 (Pin_22); no longer J1.21 (Pin_21)
- net LED_Q3: now also J1.20 (Pin_20); no longer J1.19 (Pin_19)
- net LED_Q4: now also J1.18 (Pin_18); no longer J1.17 (Pin_17)
- net LED_Q5: now also J1.16 (Pin_16); no longer J1.15 (Pin_15)
- net LED_Q6: now also J1.14 (Pin_14); no longer J1.13 (Pin_13)
- net LED_Q7: now also J1.12 (Pin_12); no longer J1.11 (Pin_11)
- net LED_Q8: now also J1.10 (Pin_10); no longer J1.9 (Pin_9)

Commit message: [HMI] Fix Q LEDs inverted + add silk labels
Connections:
- net LED_Q1: now also D9.2 (A); no longer D16.2 (A)
- net LED_Q2: now also D10.2 (A); no longer D15.2 (A)
- net LED_Q3: now also D11.2 (A); no longer D14.2 (A)
- net LED_Q4: now also D12.2 (A); no longer D13.2 (A)
- net LED_Q5: now also D13.2 (A); no longer D12.2 (A)
- net LED_Q6: now also D14.2 (A); no longer D11.2 (A)
- net LED_Q7: now also D15.2 (A); no longer D10.2 (A)
- net LED_Q8: now also D16.2 (A); no longer D9.2 (A)
Other:
- moved on the sheet: D10, D11, D12, D13, D14, D15, D16, D9
Changed lines of the file:
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@@
     )
   )
-  (symbol (lib_id "Device:LED") (at 158.75 132.08 90) (unit 1)
-    (in_bom yes) (on_board yes) (dnp no)
-    (property "Reference" "D10" (at 161.29 130.81 90)
-      (effects (font (size 1.27 1.27)) (justify right))
-    )
-    (property "Value" "Red" (at 161.29 133.35 90)
-      (effects (font (size 1.27 1.27)) (justify right))
-    )
-    (property "Footprint" "LED_THT:LED_D5.0mm" (at 158.75 132.08 0)
-      (effects (font (size 1.27 1.27)) hide)
-    )
-    (property "Datasheet" "~" (at 158.75 132.08 0)
-      (effects (font (size 1.27 1.27)) hide)
-    )
-    (property "LCSC" "C417347" (at 158.75 132.08 0)
+  (symbol (lib_id "Device:LED") (at 203.2 132.08 90) (unit 1)
+    (in_bom yes) (on_board yes) (dnp no)
+    (property "Reference" "D10" (at 205.74 130.81 90)
+      (effects (font (size 1.27 1.27)) (justify right))
+    )
+    (property "Value" "Red" (at 205.74 133.35 90)
+      (effects (font (size 1.27 1.27)) (justify right))
+    )
+    (property "Footprint" "LED_THT:LED_D5.0mm" (at 203.2 132.08 0)
+      (effects (font (size 1.27 1.27)) hide)
+    )
+    (property "Datasheet" "~" (at 203.2 132.08 0)
+      (effects (font (size 1.27 1.27)) hide)
+    )
+    (property "LCSC" "C417347" (at 203.2 132.08 0)
       (effects (font (size 1.27 1.27)) hide)
     )
@@
     )
   )
+  (symbol (lib_id "Device:LED") (at 149.86 132.08 90) (unit 1)
+    (in_bom yes) (on_board yes) (dnp no)
+    (property "Reference" "D16" (at 152.4 130.81 90)
+      (effects (font (size 1.27 1.27)) (justify right))
+    )
+    (property "Value" "Red" (at 152.4 133.35 90)
+      (effects (font (size 1.27 1.27)) (justify right))
+    )
+    (property "Footprint" "LED_THT:LED_D5.0mm" (at 149.86 132.08 0)
+      (effects (font (size 1.27 1.27)) hide)
+    )
+    (property "Datasheet" "~" (at 149.86 132.08 0)
+      (effects (font (size 1.27 1.27)) hide)
+    )
+    (property "LCSC" "C417347" (at 149.86 132.08 0)
+      (effects (font (size 1.27 1.27)) hide)
+    )
+    (pin "1")
+    (pin "2")
+    (instances
+      (project "PiPLC-HMI"
+        (path "/8e79ca85-0324-46f6-b833-7804912a961b"
+          (reference "D16") (unit 1)
+        )
+      )
+    )
+  )
   (symbol (lib_id "Device:LED") (at 212.09 132.08 90) (unit 1)
     (in_bom yes) (on_board yes) (dnp no)
-    (property "Reference" "D16" (at 214.63 130.81 90)
+    (property "Reference" "D9" (at 214.63 130.81 90)
       (effects (font (size 1.27 1.27)) (justify right))
     )
@@
     )
     (property "LCSC" "C417347" (at 212.09 132.08 0)
-      (effects (font (size 1.27 1.27)) hide)
-    )
-    (pin "1")
-    (pin "2")
-    (instances
-      (project "PiPLC-HMI"
-        (path "/8e79ca85-0324-46f6-b833-7804912a961b"
-          (reference "D16") (unit 1)
-        )
-      )
-    )
-  )
-  (symbol (lib_id "Device:LED") (at 149.86 132.08 90) (unit 1)
-    (in_bom yes) (on_board yes) (dnp no)
-    (property "Reference" "D9" (at 152.4 130.81 90)
-      (effects (font (size 1.27 1.27)) (justify right))
-    )
-    (property "Value" "Red" (at 152.4 133.35 90)
-      (effects (font (size 1.27 1.27)) (justify right))
-    )
-    (property "Footprint" "LED_THT:LED_D5.0mm" (at 149.86 132.08 0)
-      (effects (font (size 1.27 1.27)) hide)
-    )
-    (property "Datasheet" "~" (at 149.86 132.08 0)
-      (effects (font (size 1.27 1.27)) hide)
-    )
-    (property "LCSC" "C417347" (at 149.86 132.08 0)
       (effects (font (size 1.27 1.27)) hide)
     )
@@
     )
   )
-  (symbol (lib_id "Device:LED") (at 167.64 132.08 90) (unit 1)
-    (in_bom yes) (on_board yes) (dnp no)
-    (property "Reference" "D11" (at 170.18 130.81 90)
-      (effects (font (size 1.27 1.27)) (justify right))
-    )
-    (property "Value" "Red" (at 170.18 133.35 90)
-      (effects (font (size 1.27 1.27)) (justify right))
-    )
-    (property "Footprint" "LED_THT:LED_D5.0mm" (at 167.64 132.08 0)
-      (effects (font (size 1.27 1.27)) hide)
-    )
-    (property "Datasheet" "~" (at 167.64 132.08 0)
-      (effects (font (size 1.27 1.27)) hide)
-    )
-    (property "LCSC" "C417347" (at 167.64 132.08 0)
+  (symbol (lib_id "Device:LED") (at 194.31 132.08 90) (unit 1)
+    (in_bom yes) (on_board yes) (dnp no)
+    (property "Reference" "D11" (at 196.85 130.81 90)
+      (effects (font (size 1.27 1.27)) (justify right))
+    )
+    (property "Value" "Red" (at 196.85 133.35 90)
+      (effects (font (size 1.27 1.27)) (justify right))
+    )
+    (property "Footprint" "LED_THT:LED_D5.0mm" (at 194.31 132.08 0)
+      (effects (font (size 1.27 1.27)) hide)
+    )
+    (property "Datasheet" "~" (at 194.31 132.08 0)
+      (effects (font (size 1.27 1.27)) hide)
+    )
+    (property "LCSC" "C417347" (at 194.31 132.08 0)
       (effects (font (size 1.27 1.27)) hide)
     )
@@
     )
   )
-  (symbol (lib_id "Device:LED") (at 203.2 132.08 90) (unit 1)
-    (in_bom yes) (on_board yes) (dnp no)
-    (property "Reference" "D15" (at 205.74 130.81 90)
-      (effects (font (size 1.27 1.27)) (justify right))
-    )
-    (property "Value" "Red" (at 205.74 133.35 90)
-      (effects (font (size 1.27 1.27)) (justify right))
-    )
-    (property "Footprint" "LED_THT:LED_D5.0mm" (at 203.2 132.08 0)
-      (effects (font (size 1.27 1.27)) hide)
-    )
-    (property "Datasheet" "~" (at 203.2 132.08 0)
-      (effects (font (size 1.27 1.27)) hide)
-    )
-    (property "LCSC" "C417347" (at 203.2 132.08 0)
+  (symbol (lib_id "Device:LED") (at 158.75 132.08 90) (unit 1)
+    (in_bom yes) (on_board yes) (dnp no)
+    (property "Reference" "D15" (at 161.29 130.81 90)
+      (effects (font (size 1.27 1.27)) (justify right))
+    )
+    (property "Value" "Red" (at 161.29 133.35 90)
+      (effects (font (size 1.27 1.27)) (justify right))
+    )
+    (property "Footprint" "LED_THT:LED_D5.0mm" (at 158.75 132.08 0)
+      (effects (font (size 1.27 1.27)) hide)
+    )
+    (property "Datasheet" "~" (at 158.75 132.08 0)
+      (effects (font (size 1.27 1.27)) hide)
+    )
+    (property "LCSC" "C417347" (at 158.75 132.08 0)
       (effects (font (size 1.27 1.27)) hide)
     )
@@
     )
   )
+  (symbol (lib_id "Device:LED") (at 176.53 132.08 90) (unit 1)
+    (in_bom yes) (on_board yes) (dnp no)
+    (property "Reference" "D13" (at 179.07 130.81 90)
+      (effects (font (size 1.27 1.27)) (justify right))
+    )
+    (property "Value" "Red" (at 179.07 133.35 90)
+      (effects (font (size 1.27 1.27)) (justify right))
+    )
+    (property "Footprint" "LED_THT:LED_D5.0mm" (at 176.53 132.08 0)
+      (effects (font (size 1.27 1.27)) hide)
+    )
+    (property "Datasheet" "~" (at 176.53 132.08 0)
+      (effects (font (size 1.27 1.27)) hide)
+    )
+    (property "LCSC" "C417347" (at 176.53 132.08 0)
+      (effects (font (size 1.27 1.27)) hide)
+    )
+    (pin "1")
+    (pin "2")
+    (instances
+      (project "PiPLC-HMI"
+        (path "/8e79ca85-0324-46f6-b833-7804912a961b"
+          (reference "D13") (unit 1)
+        )
+      )
+    )
+  )
   (symbol (lib_id "Device:LED") (at 185.42 132.08 90) (unit 1)
     (in_bom yes) (on_board yes) (dnp no)
-    (property "Reference" "D13" (at 187.96 130.81 90)
+    (property "Reference" "D12" (at 187.96 130.81 90)
       (effects (font (size 1.27 1.27)) (justify right))
     )
@@
       (project "PiPLC-HMI"
         (path "/8e79ca85-0324-46f6-b833-7804912a961b"
-          (reference "D13") (unit 1)
-        )
-      )
-    )
-  )
-  (symbol (lib_id "Device:LED") (at 176.53 132.08 90) (unit 1)
-    (in_bom yes) (on_board yes) (dnp no)
-    (property "Reference" "D12" (at 179.07 130.81 90)
-      (effects (font (size 1.27 1.27)) (justify right))
-    )
-    (property "Value" "Red" (at 179.07 133.35 90)
-      (effects (font (size 1.27 1.27)) (justify right))
-    )
-    (property "Footprint" "LED_THT:LED_D5.0mm" (at 176.53 132.08 0)
-      (effects (font (size 1.27 1.27)) hide)
-    )
-    (property "Datasheet" "~" (at 176.53 132.08 0)
-      (effects (font (size 1.27 1.27)) hide)
-    )
-    (property "LCSC" "C417347" (at 176.53 132.08 0)
-      (effects (font (size 1.27 1.27)) hide)
-    )
-    (pin "1")
-    (pin "2")
-    (instances
-      (project "PiPLC-HMI"
-        (path "/8e79ca85-0324-46f6-b833-7804912a961b"
           (reference "D12") (unit 1)
         )
@@
     )
   )
-  (symbol (lib_id "Device:LED") (at 194.31 132.08 90) (unit 1)
-    (in_bom yes) (on_board yes) (dnp no)
-    (property "Reference" "D14" (at 196.85 130.81 90)
-      (effects (font (size 1.27 1.27)) (justify right))
-    )
-    (property "Value" "Red" (at 196.85 133.35 90)
-      (effects (font (size 1.27 1.27)) (justify right))
-    )
-    (property "Footprint" "LED_THT:LED_D5.0mm" (at 194.31 132.08 0)
-      (effects (font (size 1.27 1.27)) hide)
-    )
-    (property "Datasheet" "~" (at 194.31 132.08 0)
-      (effects (font (size 1.27 1.27)) hide)
-    )
-    (property "LCSC" "C417347" (at 194.31 132.08 0)
-      (effects (font (size 1.27 1.27)) hide)
-    )
+  (symbol (lib_id "Device:LED") (at 167.64 132.08 90) (unit 1)
+    (in_bom yes) (on_board yes) (dnp no)
+    (property "Reference" "D14" (at 170.18 130.81 90)
+      (effects (font (size 1.27 1.27)) (justify right))
+    )
+    (property "Value" "Red" (at 170.18 133.35 90)
+      (effects (font (size 1.27 1.27)) (justify right))
+    )
+    (property "Footprint" "LED_THT:LED_D5.0mm" (at 167.64 132.08 0)
+      (effects (font (size 1.27 1.27)) hide)
+    )
+    (property "Datasheet" "~" (at 167.64 132.08 0)
+      (effects (font (size 1.27 1.27)) hide)
+    )
+    (property "LCSC" "C417347" (at 167.64 132.08 0)
+      (effects (font (size 1.27 1.27)) hide)
+    )
