File: pcb/PiPLC-HMI/PiPLC-HMI.kicad_pcb (KiCad board)
At the start: 2 copper layers, 86.4 x 50 mm, 26 parts, among them J1 Conn_02x12_Odd_Even, J2 KNX

Commit message: [HMI] Add commit info and reorder
Other:
- board text added: "HMI Board 774f47b"
- board text removed: "HMI Board COMMITXY"
Changed lines of the file:
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@@
     (effects (font (size 1 1) (thickness 0.15)) (justify left bottom))
   )
-  (gr_text "HMI Board\nCOMMITXY" (at 143.554 87.882) (layer "F.SilkS")
+  (gr_text "HMI Board\n774f47b" (at 143.554 87.882) (layer "F.SilkS")
     (effects (font (size 1 1) (thickness 0.15)) (justify left bottom))
   )
